File: PCB/wakeupbro.kicad_sch (KiCad schematic)
At the start: 14 parts, among them J1 Conn_01x08_Pin, SW1 SW_Push, SW2 SW_Push, SW3 SW_Push, U1 XIAO-ESP32-C3-SMD

Commit message: Organized schematic a bit and just yea idk.
Parts:
- BZ1: footprint (none) -> Buzzer_Beeper:Buzzer_12x9.5RM7.6
- H1, H2, H3, H4: footprint (none) -> MountingHole:MountingHole_3.2mm_M3
- J1: footprint (none) -> Connector_PinSocket_2.54mm:PinSocket_1x08_P2.54mm_Vertical
- SW1, SW2, SW3: footprint (none) -> Button_Switch_Keyboard:SW_Cherry_MX_1.00u_PCB
Other:
- note added: "Display"
- note added: "LEDs(Extras from hackpad)"
- note added: "le microcontroler =D"
- note added: "the big three switches =D"
- title: (none) -> wake up bro
- moved on the sheet: BZ1, D1, D2, D3, D4, J1, SW1, SW2, SW3, U1

Commit message: Routed PCB, silkscreen art soon...
Parts:
- D1, D2, D3, D4: footprint LED_SMD:LED_SK6812MINI_PLCC4_3.5x3.5mm_P1.75mm -> LED_SMD:LED_SK6812MINI-E_3.2x2.8mm_P1.5mm_ReverseMount
- U1: footprint Seeed_Studio_XIAO_Series:XIAO-ESP32-C3-SMD -> Seeed_Studio_XIAO_Series:XIAO-ESP32-C3-DIP
Connections:
- net LED renamed DIN
Changed lines of the file:
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@@
 		)
 	)
-	(global_label "LED"
+	(global_label "DIN"
 		(shape input)
 		(at 140.97 140.97 180)
@@
 		)
 		(property "Intersheetrefs" "${INTERSHEET_REFS}"
-			(at 134.5377 140.97 0)
+			(at 134.7795 140.97 0)
 			(hide yes)
 			(show_name no)
@@
 		)
 	)
-	(global_label "LED"
+	(global_label "DIN"
 		(shape input)
 		(at 115.57 52.07 180)
@@
 		)
 		(property "Intersheetrefs" "${INTERSHEET_REFS}"
-			(at 109.1377 52.07 0)
+			(at 109.3795 52.07 0)
 			(hide yes)
 			(show_name no)
@@
 			)
 		)
-		(property "Footprint" "LED_SMD:LED_SK6812MINI_PLCC4_3.5x3.5mm_P1.75mm"
+		(property "Footprint" "LED_SMD:LED_SK6812MINI-E_3.2x2.8mm_P1.5mm_ReverseMount"
 			(at 184.15 148.59 0)
 			(hide yes)
@@
 			)
 		)
-		(property "Footprint" "LED_SMD:LED_SK6812MINI_PLCC4_3.5x3.5mm_P1.75mm"
+		(property "Footprint" "LED_SMD:LED_SK6812MINI-E_3.2x2.8mm_P1.5mm_ReverseMount"
 			(at 212.09 148.59 0)
 			(hide yes)
@@
 			)
 		)
-		(property "Footprint" "Seeed_Studio_XIAO_Series:XIAO-ESP32-C3-SMD"
+		(property "Footprint" "Seeed_Studio_XIAO_Series:XIAO-ESP32-C3-DIP"
 			(at 101.092 84.074 0)
 			(hide yes)
@@
 			)
 		)
-		(property "Footprint" "LED_SMD:LED_SK6812MINI_PLCC4_3.5x3.5mm_P1.75mm"
+		(property "Footprint" "LED_SMD:LED_SK6812MINI-E_3.2x2.8mm_P1.5mm_ReverseMount"
 			(at 238.76 148.59 0)
 			(hide yes)
@@
 			)
 		)
-		(property "Footprint" "LED_SMD:LED_SK6812MINI_PLCC4_3.5x3.5mm_P1.75mm"
+		(property "Footprint" "LED_SMD:LED_SK6812MINI-E_3.2x2.8mm_P1.5mm_ReverseMount"
 			(at 157.48 148.59 0)
 			(hide yes)

Commit message: Update PCB files. Going to start workig on firmware
Parts:
- D1, D2, D3, D4: footprint LED_SMD:LED_SK6812MINI-E_3.2x2.8mm_P1.5mm_ReverseMount -> footprints:SK6812MINI-E_fixed
Changed lines of the file:
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@@
 			)
 		)
-		(property "Footprint" "LED_SMD:LED_SK6812MINI-E_3.2x2.8mm_P1.5mm_ReverseMount"
+		(property "Footprint" "footprints:SK6812MINI-E_fixed"
 			(at 184.15 148.59 0)
 			(hide yes)
@@
 			)
 		)
-		(property "Footprint" "LED_SMD:LED_SK6812MINI-E_3.2x2.8mm_P1.5mm_ReverseMount"
+		(property "Footprint" "footprints:SK6812MINI-E_fixed"
 			(at 212.09 148.59 0)
 			(hide yes)
@@
 			)
 		)
-		(property "Footprint" "LED_SMD:LED_SK6812MINI-E_3.2x2.8mm_P1.5mm_ReverseMount"
+		(property "Footprint" "footprints:SK6812MINI-E_fixed"
 			(at 238.76 148.59 0)
 			(hide yes)
@@
 			)
 		)
-		(property "Footprint" "LED_SMD:LED_SK6812MINI-E_3.2x2.8mm_P1.5mm_ReverseMount"
+		(property "Footprint" "footprints:SK6812MINI-E_fixed"
 			(at 157.48 148.59 0)
 			(hide yes)
